File: p9660/p9660.kicad_sch (KiCad schematic)
At the start: 1 part

Commit message: Design probably works ™️
Parts:
- added J1, J2, J3, J4: Conn_02x08_Counter_Clockwise, Connector_PinHeader_2.54mm:PinHeader_2x08_P2.54mm_Vertical, symbol Connector_Generic:Conn_02x08_Odd_Even
- added J5: Conn_02x04_Counter_Clockwise, Connector_PinHeader_2.54mm:PinHeader_2x04_P2.54mm_Horizontal, symbol Connector_Generic:Conn_02x04_Odd_Even
Connections:
- net D0: now also J1.1 (Pin_1); no longer C1.12 (D13), C1.15 (D17), C1.18 (D21), C1.21 (CK2+), C1.24 (D27), C1.27 (D31), C1.3 (D3), C1.31 (D4), C1.34 (CK1+), C1.37 (D10), C1.40 (D14), C1.43 (D18), C1.46 (D22), C1.49 (D24), C1.52 (D28), C1.6 (D7), C1.9 (D9)
- net D1: now also J1.3 (Pin_3); no longer C1.11 (D12), C1.14 (D16), C1.17 (D20), C1.2 (D2), C1.20 (CK2-), C1.23 (D26), C1.26 (D30), C1.32 (D5), C1.35 (CK1-), C1.38 (D11), C1.41 (D15), C1.44 (D19), C1.47 (D23), C1.5 (D6), C1.50 (D25), C1.53 (D29), C1.8 (D8)
- net GND: now also J1.10 (Pin_10), J1.12 (Pin_12), J1.14 (Pin_14), J1.16 (Pin_16), J1.2 (Pin_2), J1.4 (Pin_4), J1.6 (Pin_6), J1.8 (Pin_8), J2.10 (Pin_10), J2.12 (Pin_12), J2.14 (Pin_14), J2.16 (Pin_16), J2.2 (Pin_2), J2.4 (Pin_4), J2.6 (Pin_6), J2.8 (Pin_8), J3.10 (Pin_10), J3.12 (Pin_12), J3.14 (Pin_14), J3.16 (Pin_16), J3.2 (Pin_2), J3.4 (Pin_4), J3.6 (Pin_6), J3.8 (Pin_8), J4.10 (Pin_10), J4.12 (Pin_12), J4.14 (Pin_14), J4.16 (Pin_16), J4.2 (Pin_2), J4.4 (Pin_4), J4.6 (Pin_6), J4.8 (Pin_8), J5.1 (Pin_1), J5.2 (Pin_2), J5.7 (Pin_7), J5.8 (Pin_8)
- new net CK1+: C1.34 (CK1+), J5.3 (Pin_3)
- new net CK1-: C1.35 (CK1-), J5.5 (Pin_5)
- new net CK2+: C1.21 (CK2+), J5.6 (Pin_6)
- new net CK2-: C1.20 (CK2-), J5.4 (Pin_4)
- new net D10: C1.37 (D10), J2.5 (Pin_5)
- new net D11: C1.38 (D11), J2.7 (Pin_7)
- new net D12: C1.11 (D12), J2.9 (Pin_9)
- new net D13: C1.12 (D13), J2.11 (Pin_11)
- new net D14: C1.40 (D14), J2.13 (Pin_13)
- new net D15: C1.41 (D15), J2.15 (Pin_15)
- new net D16: C1.14 (D16), J3.1 (Pin_1)
- new net D17: C1.15 (D17), J3.3 (Pin_3)
- new net D18: C1.43 (D18), J3.5 (Pin_5)
- new net D19: C1.44 (D19), J3.7 (Pin_7)
- new net D2: C1.2 (D2), J1.5 (Pin_5)
- new net D20: C1.17 (D20), J3.9 (Pin_9)
- new net D21: C1.18 (D21), J3.11 (Pin_11)
- new net D22: C1.46 (D22), J3.13 (Pin_13)
- new net D23: C1.47 (D23), J3.15 (Pin_15)
- new net D24: C1.49 (D24), J4.1 (Pin_1)
- new net D25: C1.50 (D25), J4.3 (Pin_3)
- new net D26: C1.23 (D26), J4.5 (Pin_5)
- new net D27: C1.24 (D27), J4.7 (Pin_7)
- new net D28: C1.52 (D28), J4.9 (Pin_9)
- new net D29: C1.53 (D29), J4.11 (Pin_11)
- new net D3: C1.3 (D3), J1.7 (Pin_7)
- new net D30: C1.26 (D30), J4.13 (Pin_13)
- new net D31: C1.27 (D31), J4.15 (Pin_15)
- new net D4: C1.31 (D4), J1.9 (Pin_9)
- new net D5: C1.32 (D5), J1.11 (Pin_11)
- new net D6: C1.5 (D6), J1.13 (Pin_13)
- new net D7: C1.6 (D7), J1.15 (Pin_15)
- new net D8: C1.8 (D8), J2.1 (Pin_1)
- new net D9: C1.9 (D9), J2.3 (Pin_3)

Commit message: done for realz?
Parts:
- added TP1, TP2, TP3, TP4, TP5, TP6, TP7, TP8: TestPoint, TestPoint:TestPoint_Pad_2.0x2.0mm, symbol Connector:TestPoint
Connections:
- net GND: now also TP1.1, TP2.1, TP3.1, TP4.1, TP5.1, TP6.1, TP7.1, TP8.1
