File: kicad/p6960.kicad_pcb (KiCad board)
At the start: 2 copper layers, 58 x 51 mm, 15 parts, among them J1 Conn_02x08_Counter_Clockwise, J2 Conn_02x08_Counter_Clockwise, J3 Conn_02x08_Counter_Clockwise, J4 Conn_02x08_Counter_Clockwise, J5 Conn_02x04_Counter_Clockwise

Commit message: fix my mild dyslexia
Other:
- board text added: "github.com/hadn69/P69xx-Breakout"
- board text removed: "github.com/hadn69/P9660-Breakout"

Commit message: tuned trace lengths
Parts:
- C1: footprint Tek:P9660 -> Tek:P69xx
- moved J3 3.34 mm to (88.9, 34.6)
- moved J1 3.10 mm to (49.4, 34.6)
- moved J2 3.10 mm to (49.4, 56.6)
- moved J4 2.94 mm to (88.9, 56.5)
Connections:
- C1 pad 2: GND -> D2
- C1 pad 3: GND -> D3
Routing:
- net GND: track 153.5 -> 0.00 mm, vias 27 -> 29
- net D14: track 40.7 -> 28.7 mm
- net D17: track 40.7 -> 28.7 mm
- net D8: track 38.4 -> 28.7 mm
- net D23: track 38.4 -> 28.7 mm
- net D18: track 38.2 -> 28.7 mm
- net D13: track 38.2 -> 28.7 mm
- net D22: track 34.9 -> 28.7 mm
- net D9: track 34.9 -> 28.7 mm
- net D10: track 34.8 -> 28.6 mm
- net D21: track 34.8 -> 28.6 mm
- net D11: track 34.8 -> 28.7 mm
- net D20: track 34.8 -> 28.7 mm
- net D15: track 34.8 -> 28.8 mm
- net D16: track 34.8 -> 28.8 mm
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